File: bizcard/bizcard.kicad_sch (KiCad schematic)
At the start: 0 parts

Commit message: Push
Other:
- removed sheet usb
- sheet micro ports: added LED_DOUT; removed none
Changed lines of the file:
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@@
 	(generator_version "8.0")
 	(paper "A4")
-	(sheet
-		(at 52.07 64.77)
-		(size 34.29 30.48)
-		(fields_autoplaced yes)
+	(wire
+		(pts
+			(xy 121.92 71.12) (xy 137.16 71.12)
+		)
 		(stroke
-			(width 0.1524)
-			(type solid)
-		)
-		(fill
-			(color 0 0 0 0.0000)
-		)
-		(property "Sheetname" "usb"
-			(at 52.07 64.0584 0)
-			(effects
-				(font
-					(size 1.27 1.27)
-				)
-				(justify left bottom)
-			)
-		)
-		(property "Sheetfile" "usb.kicad_sch"
-			(at 52.07 95.8346 0)
-			(effects
-				(font
-					(size 1.27 1.27)
-				)
-				(justify left top)
-			)
-		)
-		(instances
-			(project "bizcard"
-				(path "/7f3f26e1-61db-49d8-a68c-f315156bfd80"
-					(page "3")
-				)
-			)
+			(width 0)
+			(type default)
 		)
 	)
 	(sheet
-		(at 204.47 63.5)
+		(at 137.16 68.58)
 		(size 20.32 4.445)
 		(fields_autoplaced yes)
@@
 		)
 		(property "Sheetname" "led"
-			(at 204.47 62.7884 0)
+			(at 137.16 67.8684 0)
 			(effects
 				(font
@@
 		)
 		(property "Sheetfile" "led.kicad_sch"
-			(at 204.47 68.5296 0)
+			(at 137.16 73.6096 0)
 			(effects
 				(font
@@
 		)
 		(pin "DIN" input
-			(at 204.47 66.04 180)
+			(at 137.16 71.12 180)
 			(effects
 				(font
@@
 	)
 	(sheet
-		(at 124.46 63.5)
-		(size 44.45 31.75)
+		(at 95.25 68.58)
+		(size 26.67 5.715)
 		(fields_autoplaced yes)
 		(stroke
@@
 		)
 		(property "Sheetname" "micro"
-			(at 124.46 62.7884 0)
+			(at 95.25 67.8684 0)
 			(effects
 				(font
@@
 		)
 		(property "Sheetfile" "micro.kicad_sch"
-			(at 124.46 95.8346 0)
+			(at 95.25 74.8796 0)
 			(effects
 				(font
@@
 			)
 		)
+		(pin "LED_DOUT" output
+			(at 121.92 71.12 0)
+			(effects
+				(font
+					(size 1.27 1.27)
+				)
+				(justify right)
+			)
+		)
