File: bizcard/bizcard.kicad_pcb (KiCad board)
At the start: 2 copper layers, 82 x 53.5 mm, 204 parts, among them J1 Conn_01x06_Pin, U1 MCP1700T-3302E_TT, U2 STM32F042K6Tx

Commit message: Sync
Parts:
- C12, C13, C14, C15, C16, C17, C18, C19, C20, C21, C34, C35, C40, C41, C42, C43, C44, C45, R12, R13, R14, R15, R16, R17, R18, R19, R20, R21, R22, R23, R24, R25, R26, R27, R28, R29, R30, R31, R56, R57, R58, R59, R68, R69, R70, R71, R72, R73, R74, R75, R76, R77, R78, R79, U10, U11, U12, U13, U14, U27, U28, U33, U34, U35, U36, U37, U38, U5, U6, U7, U8, U9: moved to B.Cu
- moved R68 123.6 mm to (114.0, 102.2), turned to 180 degrees
- moved R69 119.4 mm to (116.5, 100.5), turned to 90 degrees
- moved U33 117.8 mm to (114.3, 99.2)
- moved C40 112.3 mm to (116.5, 98.5), turned to 90 degrees
- moved R58 108.3 mm to (117.0, 96.5), turned to 180 degrees
- moved R59 107.2 mm to (117.0, 92.2), turned to -90 degrees
- moved R70 104.9 mm to (118.5, 101.8), turned to 180 degrees
- moved C35 102.4 mm to (116.5, 94.2), turned to -90 degrees
- moved R71 101.6 mm to (121.5, 100.5), turned to 90 degrees
- moved U28 101.6 mm to (119.4, 93.8)
- moved U34 100.2 mm to (119.2, 99.2)
- moved R20 99.1 mm to (113.8, 69.0), turned to 90 degrees
- moved C41 96.2 mm to (121.5, 98.5), turned to 90 degrees
- moved R21 94.4 mm to (118.5, 70.5), turned to 90 degrees
- moved R26 94.0 mm to (129.8, 68.2), turned to 180 degrees
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Routing:
- net GND: track 2.17 -> 41.7 mm
- net +5V: track 1.10 -> 39.8 mm, vias 0 -> 8
- net Net-(D9-G-): track 0.00 -> 14.2 mm, vias 0 -> 1
- net Net-(D10-G-): track 0.00 -> 14.1 mm, vias 0 -> 1
- net Net-(D16-G-): track 0.00 -> 13.1 mm, vias 0 -> 3
- net Net-(D8-G-): track 0.00 -> 12.9 mm, vias 0 -> 1
- net Net-(D10-R-): track 0.00 -> 12.7 mm, vias 0 -> 1
- net Net-(D9-R-): track 0.00 -> 12.6 mm, vias 0 -> 1
- net Net-(D35-G-): track 0.00 -> 12.6 mm, vias 0 -> 1
- net Net-(D16-R-): track 0.00 -> 12.0 mm, vias 0 -> 1
- net Net-(D35-R-): track 0.00 -> 11.9 mm, vias 0 -> 1
- net Net-(D10-B-): track 0.00 -> 11.6 mm, vias 0 -> 1
- net Net-(D40-G-): track 0.00 -> 11.6 mm, vias 0 -> 1
- net Net-(D40-R-): track 0.00 -> 11.5 mm, vias 0 -> 1
- net Net-(D7-G-): track 0.00 -> 11.5 mm, vias 0 -> 1
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Other:
- board size 82 x 53.5 mm -> 82 x 52.5 mm

Commit message: zoop
Parts:
- C36, C37, C38, C39, R60, R61, R62, R63, R64, R65, R66, R67, U29, U30, U31, U32: moved to B.Cu
- moved R60 99.8 mm to (121.5, 96.2), turned to 180 degrees
- moved R62 97.3 mm to (126.5, 96.2), turned to 180 degrees
- moved R61 97.3 mm to (121.8, 92.2), turned to -90 degrees
- moved R63 96.9 mm to (126.2, 92.2), turned to -90 degrees
- moved U29 92.6 mm to (124.0, 93.8)
- moved C36 92.1 mm to (121.8, 94.2), turned to -90 degrees
- moved C37 91.7 mm to (126.2, 94.2), turned to -90 degrees
- moved U30 91.0 mm to (128.8, 93.8)
- moved R64 57.9 mm to (131.0, 96.2), turned to 180 degrees
- moved R65 53.8 mm to (131.0, 92.2), turned to -90 degrees
- moved U31 50.9 mm to (133.2, 93.8)
- moved C38 49.3 mm to (131.0, 94.2), turned to -90 degrees
- moved R67 36.8 mm to (135.5, 92.5), turned to -90 degrees
- moved R66 36.6 mm to (136.0, 96.2), turned to 180 degrees
- moved C39 31.6 mm to (135.5, 94.8), turned to -90 degrees
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Routing:
- net Net-(D34-R-): track 0.00 -> 9.22 mm, vias 0 -> 1
- net Net-(D34-G-): track 0.00 -> 9.21 mm, vias 0 -> 1
- net Net-(D33-G-): track 0.00 -> 8.80 mm, vias 0 -> 1
- net Net-(D32-G-): track 0.00 -> 8.40 mm, vias 0 -> 1
- net Net-(D33-R-): track 0.00 -> 8.35 mm, vias 0 -> 1
- net Net-(D34-B-): track 0.00 -> 8.27 mm, vias 0 -> 1
- net GND: track 41.7 -> 49.7 mm
- net Net-(D32-R-): track 0.00 -> 7.92 mm, vias 0 -> 1
- net Net-(D33-B-): track 0.00 -> 7.49 mm, vias 0 -> 1
- net Net-(D31-G-): track 0.00 -> 7.46 mm, vias 0 -> 1
- net Net-(D31-R-): track 0.00 -> 7.02 mm, vias 0 -> 1
- net Net-(D32-B-): track 0.00 -> 6.89 mm, vias 0 -> 1
- net Net-(D31-B-): track 0.00 -> 6.17 mm, vias 0 -> 1
- net Net-(U29-DIN): track 0.00 -> 3.18 mm
- net Net-(U30-DIN): track 0.00 -> 3.04 mm
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
Commit message: Margin rules
Parts:
- C22, C23, C24, C25, C26, C27, C28, C29, C30, C31, C32, C33, D3, R32, R33, R34, R35, R36, R37, R38, R39, R40, R41, R42, R43, R44, R45, R46, R47, R48, R49, R50, R51, R52, R53, R54, R55, U15, U16, U17, U18, U19, U20, U21, U22, U23, U24, U25, U26: moved to B.Cu
- moved D3 118.2 mm to (81.0, 69.5), turned to 45 degrees
- moved R44 105.3 mm to (109.2, 83.8), turned to 90 degrees
- moved R40 104.2 mm to (129.8, 82.8), turned to 180 degrees
- moved R33 102.4 mm to (108.8, 78.5), turned to 90 degrees
- moved R50 99.7 mm to (125.8, 87.0), turned to 180 degrees
- moved R45 99.0 mm to (115.2, 83.5), turned to 180 degrees
- moved U21 98.7 mm to (112.0, 83.8), turned to 180 degrees
- moved R35 98.4 mm to (114.5, 78.5), turned to 90 degrees
- moved R32 98.4 mm to (112.0, 74.0)
- moved R34 98.0 mm to (115.0, 76.0), turned to 180 degrees
- moved U19 97.4 mm to (131.7, 80.2)
- moved R41 97.2 mm to (135.0, 79.5), turned to -90 degrees
- moved U15 95.9 mm to (112.0, 77.8), turned to 180 degrees
- moved C22 95.5 mm to (109.8, 78.5), turned to -90 degrees
- moved R51 94.3 mm to (130.2, 84.5), turned to -90 degrees
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Routing:
- net Net-(D28-B-): track 0.00 -> 8.85 mm, vias 0 -> 1
- net Net-(D27-B-): track 0.00 -> 8.59 mm, vias 0 -> 1
- net Net-(D17-G-): track 0.00 -> 8.34 mm, vias 0 -> 1
- net Net-(D17-B-): track 0.00 -> 8.18 mm, vias 0 -> 1
- net Net-(D28-G-): track 0.00 -> 7.68 mm, vias 0 -> 1
- net GND: track 49.7 -> 57.4 mm
- net Net-(D23-B-): track 0.00 -> 6.64 mm, vias 0 -> 1
- net /led/ledsub_23/DOUT: track 0.00 -> 6.25 mm
- net Net-(D22-B-): track 0.00 -> 6.15 mm, vias 0 -> 1
- net Net-(D22-G-): track 0.00 -> 6.01 mm, vias 0 -> 1
- net Net-(U19-VDD): track 0.00 -> 5.82 mm
- net Net-(D27-G-): track 0.00 -> 5.67 mm, vias 0 -> 1
- net Net-(D21-B-): track 0.00 -> 5.61 mm, vias 0 -> 1
- net Net-(D23-G-): track 0.00 -> 5.57 mm, vias 0 -> 1
- net Net-(D22-R-): track 0.00 -> 5.51 mm, vias 0 -> 1
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
Commit message: Pop
Parts:
- U1: moved to B.Cu
- moved U1 119.7 mm to (80.0, 76.2), turned to -135 degrees
- moved J1 90.4 mm to (87.6, 63.0), turned to 90 degrees
- moved R6 3.89 mm to (82.5, 66.0)
- moved R4 3.46 mm to (79.2, 69.2)
- moved R5 3.46 mm to (80.7, 67.7)
- moved R3 3.39 mm to (77.4, 70.9)
- moved D3 2.76 mm to (83.0, 71.4)
- moved U2 2.02 mm to (88.4, 76.8), turned to 135 degrees
Routing:
- net Net-(J2-GND): track 0.00 -> 12.2 mm
- net Net-(J2-VBUS): track 0.00 -> 12.1 mm
- net Net-(J2-DP): track 0.00 -> 11.7 mm
- net Net-(J2-DM): track 1.01 -> 11.7 mm
- net +5V: track 40.8 -> 47.7 mm, vias 8 -> 9
- net GND: track 57.4 -> 63.8 mm, vias 0 -> 1
- net /micro/USB_DM: track 0.00 -> 2.87 mm
- net /micro/USB_DP: track 0.00 -> 2.42 mm
- net Net-(D3-Pad3): track 3.02 -> 2.37 mm
- net Net-(D3-Pad1): track 3.02 -> 2.44 mm

Commit message: Shift
Parts:
- C37: renamed from C2; moved to B.Cu
- C38: renamed from C4; moved to B.Cu
- C39: renamed from C3; moved to B.Cu
- C40: renamed from C6; moved to B.Cu
- C41: renamed from C7; moved to B.Cu
- C42: renamed from C8; moved to B.Cu
- C43: renamed from C9; moved to B.Cu
- C44: renamed from C1; moved to B.Cu
- moved C37 108.3 mm to (77.1, 73.7), turned to 45 degrees
- moved C39 107.1 mm to (77.8, 74.5), turned to 45 degrees
- moved C38 104.4 mm to (81.8, 78.6), turned to -45 degrees
- moved C41 104.1 mm to (94.5, 76.9), turned to 45 degrees
- moved C44 101.7 mm to (75.8, 73.2), turned to 45 degrees
- moved C42 100.3 mm to (81.9, 74.4), turned to 135 degrees
- moved C43 92.4 mm to (92.6, 81.4), turned to -45 degrees
- moved C40 90.0 mm to (95.3, 77.5), turned to 45 degrees
- moved R1 7.20 mm to (123.2, 51.2)
- renumbered C5 to C1, C19 to C10, C20 to C11, C21 to C12, C22 to C13, C23 to C14, C24 to C15, C25 to C16, C26 to C17, C27 to C18, C28 to C19, C11 to C2, C29 to C20, C30 to C21, C31 to C22, C32 to C23, C33 to C24, C34 to C25, C35 to C26, C36 to C27, C37 to C28, C38 to C29, C12 to C3, C39 to C30, C40 to C31, C41 to C32, C42 to C33, C43 to C34, C44 to C35, C45 to C36, C13 to C4, C10 to C45, C14 to C5, C15 to C6, C16 to C7, C17 to C8, C18 to C9, D6 to D1, D14 to D10, D15 to D11, D16 to D12, D17 to D13, D18 to D14, D19 to D15, D20 to D16, D21 to D17, D22 to D18, D23 to D19, D1 to D2, D24 to D20, D25 to D21, D26 to D22, D27 to D23, D28 to D24, D29 to D25, D30 to D26, D31 to D27, D32 to D28, D33 to D29, D7 to D3, D34 to D30, D35 to D31, D36 to D32, D37 to D33, D38 to D34, D39 to D35, D40 to D36, D3 to D37, D2 to D38, D4 to D39, D8 to D4, D5 to D40, D9 to D5, D10 to D6, D11 to D7, D12 to D8, D13 to D9, J2 to J1, J1 to J2, R17 to R10, R18 to R11, R19 to R12, R20 to R13, R21 to R14, R22 to R15, R23 to R16, R24 to R17, R25 to R18, R26 to R19, R27 to R20, R28 to R21, R29 to R22, R30 to R23, R31 to R24, R32 to R25, R33 to R26, R34 to R27, R35 to R28, R36 to R29, R10 to R3, R37 to R30, R38 to R31, R39 to R32, R40 to R33, R41 to R34, R42 to R35, R43 to R36, R44 to R37, R45 to R38, R46 to R39, R11 to R4, R47 to R40, R48 to R41, R49 to R42, R50 to R43, R51 to R44, R52 to R45, R53 to R46, R54 to R47, R55 to R48, R56 to R49, R12 to R5, R57 to R50, R58 to R51, R59 to R52, R60 to R53, R61 to R54, R62 to R55, R63 to R56, R64 to R57, R65 to R58, R66 to R59, R13 to R6, R67 to R60, R68 to R61, R69 to R62, R70 to R63, R71 to R64, R72 to R65, R73 to R66, R74 to R67, R75 to R68, R76 to R69, R14 to R7, R77 to R70, R78 to R71, R79 to R72, R7 to R73, R3 to R74, R4 to R75, R5 to R76, R6 to R77, R8 to R78, R9 to R79, R15 to R8, R16 to R9, U12 to U10, U13 to U11, U14 to U12, U15 to U13, U16 to U14, U17 to U15, U18 to U16, U19 to U17, U20 to U18, U21 to U19, U4 to U2, U22 to U20, U23 to U21, U24 to U22, U25 to U23, U26 to U24, U27 to U25, U28 to U26, U29 to U27, U30 to U28, U31 to U29, U5 to U3, U32 to U30, U33 to U31, U34 to U32, U35 to U33, U36 to U34, U37 to U35, U38 to U36, U2 to U37, U3 to U38, U6 to U4, U7 to U5, U8 to U6, U9 to U7, U10 to U8, U11 to U9
Routing:
- net GND: track 63.8 -> 74.8 mm
- net +3.3V: track 0.00 -> 9.87 mm
- net +5V: track 47.7 -> 53.2 mm
- net Net-(U9-DIN): track 0.00 -> 1.42 mm

Commit message: new DRC
Parts:
- C1, D2, D38, D39, R1, R2, R73: moved to B.Cu
- moved D2 121.7 mm to (75.1, 81.0), turned to 45 degrees
- moved D38 119.8 mm to (76.8, 82.6), turned to 45 degrees
- moved R2 99.8 mm to (79.0, 80.4), turned to -135 degrees
- moved D39 97.2 mm to (96.0, 69.7), turned to -135 degrees
- moved C1 94.3 mm to (93.2, 80.8), turned to -45 degrees
- moved R73 77.9 mm to (93.8, 71.9), turned to 45 degrees
- moved R1 53.6 mm to (77.3, 78.8), turned to -135 degrees
- moved C10 2.06 mm to (130.4, 67.7)
- moved C11 2.06 mm to (135.7, 68.9)
- moved C12 2.06 mm to (139.9, 67.9)
- moved C16 2.06 mm to (126.0, 77.9)
- moved C17 2.06 mm to (131.9, 79.7)
- moved C18 2.06 mm to (137.9, 79.7)
- moved C23 2.06 mm to (133.7, 85.2)
- moved C30 2.06 mm to (133.4, 94.9)
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Routing:
- net /led/DIN: track 0.00 -> 36.2 mm, vias 0 -> 2
- net +5V: track 53.2 -> 59.3 mm, vias 9 -> 12
- net +3.3V: track 9.87 -> 12.4 mm
- net Net-(U37-PB6): track 0.00 -> 2.30 mm
- net /micro/RST: track 0.00 -> 1.64 mm
- net Net-(D39-A): track 0.00 -> 1.50 mm
- net Net-(D38-A): track 0.00 -> 1.50 mm
- net Net-(D2-A): track 0.00 -> 1.44 mm
- added copper zone on F.Cu, net +5V
- added copper zone on B.Cu, net GND
Other:
- board size 82 x 52.5 mm -> 79.6 x 52.5 mm

Commit message: dru
Parts:
- moved R25 4.59 mm to (111.4, 69.8)
- moved R13 2.21 mm to (113.8, 68.5), turned to 0 degrees
- moved R17 1.98 mm to (125.2, 67.5), turned to 0 degrees
- moved C10 1.73 mm to (131.1, 69.2), turned to -90 degrees
- moved R21 1.70 mm to (134.0, 67.7), turned to 0 degrees
- moved R20 1.40 mm to (130.8, 71.5)
- moved R19 1.22 mm to (128.9, 68.2), turned to 0 degrees
- moved R15 1.10 mm to (119.3, 68.5), turned to 0 degrees
- moved C9 1.00 mm to (126.2, 69.4), turned to -90 degrees
- moved R29 1.00 mm to (120.5, 77.9), turned to 180 degrees
- moved R18 0.99 mm to (126.2, 71.4)
- moved C8 0.91 mm to (121.3, 69.5), turned to -90 degrees
- moved R16 0.86 mm to (121.3, 71.5)
- moved R14 0.76 mm to (116.5, 71.4)
- moved C7 0.73 mm to (116.4, 69.4), turned to -90 degrees
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Connections:
- R13 pad 2: /led/ledsub_6/DOUT -> /led/ledsub_7/DIN
- R15 pad 2: /led/ledsub_7/DOUT -> /led/ledsub_8/DIN
- R17 pad 2: /led/ledsub_8/DOUT -> /led/ledsub_10/DOUT
- R21 pad 2: /led/ledsub_10/DOUT -> /led/ledsub_11/DIN
- R23 pad 2: /led/ledsub_11/DOUT -> /led/ledsub_12/DIN
- R25 pad 2: /led/ledsub_12/DOUT -> /led/ledsub_13/DIN
- U11 pad 5: /led/ledsub_11/DOUT -> /led/ledsub_10/DIN
- U12 pad 5: /led/ledsub_12/DOUT -> /led/ledsub_11/DIN
- U6 pad 5: /led/ledsub_6/DOUT -> /led/ledsub_12/DIN
- U7 pad 5: /led/ledsub_7/DOUT -> /led/ledsub_13/DIN
- U8 pad 5: /led/ledsub_8/DOUT -> /led/ledsub_7/DIN
- U9 pad 5: /led/ledsub_10/DIN -> /led/ledsub_8/DIN
Routing:
- net GND: track 74.8 -> 103.9 mm, vias 1 -> 6
- net +5V: track 59.3 -> 83.5 mm, vias 12 -> 21
- net /led/ledsub_14/DOUT: track 0.00 -> 8.01 mm
- net /led/ledsub_12/DIN: track 0.00 -> 8.00 mm, vias 0 -> 2
- net Net-(U13-DIN): track 0.00 -> 7.41 mm
- net Net-(U16-DIN): track 0.00 -> 7.35 mm
- net /led/ledsub_13/DOUT: track 0.00 -> 5.06 mm
- net /led/ledsub_7/DIN: track 0.00 -> 4.42 mm
- net /led/ledsub_10/DIN: track 0.00 -> 3.91 mm
- net /led/ledsub_11/DIN: track 0.00 -> 3.91 mm
- net /led/ledsub_8/DIN: track 0.00 -> 3.57 mm
- net Net-(U14-DIN): track 0.00 -> 3.30 mm
- net /led/ledsub_10/DOUT: track 0.00 -> 3.21 mm
- net Net-(U11-DIN): track 0.00 -> 2.13 mm
- net Net-(U7-DIN): track 0.00 -> 1.35 mm
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
Commit message: zirp
Parts:
- moved R26 5.06 mm to (110.2, 75.0), turned to -90 degrees
- moved C13 5.04 mm to (111.2, 75.0), turned to 90 degrees
- moved R32 1.75 mm to (127.7, 77.0)
- moved C15 1.40 mm to (122.5, 78.0), turned to 180 degrees
- moved R28 0.85 mm to (112.5, 77.8), turned to -90 degrees
- moved C16 0.78 mm to (126.8, 77.9), turned to 180 degrees
- moved R30 0.67 mm to (124.0, 77.5), turned to -90 degrees
- moved R29 0.50 mm to (120.0, 77.9)
- moved C11 0.29 mm to (136.1, 69.1)
- moved R22 0.16 mm to (135.8, 71.2)
Routing:
- net +5V: track 83.5 -> 105.5 mm, vias 21 -> 26
- net Net-(U16-VDD): track 1.02 -> 9.31 mm, vias 0 -> 2
- net GND: track 103.9 -> 111.6 mm
- net Net-(U13-VDD): track 0.00 -> 2.23 mm
- net Net-(D7-G-): track 6.59 -> 7.45 mm
- net Net-(D12-B-): track 10.4 -> 11.1 mm
- net /led/ledsub_14/DOUT: track 8.01 -> 7.51 mm
