File: bizcard/bizcard.kicad_pcb (KiCad board)
At the start: 2 copper layers, 79.6 x 52.5 mm, 204 parts, among them J2 Conn_01x06_Pin, U1 MCP1700T-3302E_TT, U37 STM32F042K6Tx

Commit message: more
Parts:
- moved C19 6.48 mm to (107.1, 82.7)
- moved R37 6.27 mm to (113.2, 82.2), turned to 0 degrees
- moved R38 6.09 mm to (107.1, 83.7), turned to 0 degrees
- moved R47 4.13 mm to (139.3, 84.4), turned to 90 degrees
- moved R43 4.13 mm to (127.7, 86.0), turned to 0 degrees
- moved R39 2.32 mm to (113.8, 84.4), turned to -90 degrees
- moved R45 1.47 mm to (131.9, 88.2), turned to -90 degrees
- moved R41 1.34 mm to (122.2, 87.1), turned to 0 degrees
- moved C21 1.26 mm to (118.8, 86.2)
- moved R42 1.25 mm to (118.8, 87.2)
- moved C22 0.35 mm to (127.2, 84.3)
- moved R44 0.30 mm to (128.2, 84.3)
- moved R33 0.25 mm to (127.7, 82.7)
Connections:
- R37 pad 2: /led/ledsub_18/DOUT -> /led/ledsub_19/DIN
- R39 pad 2: /led/ledsub_19/DOUT -> /led/ledsub_20/DIN
- R41 pad 2: /led/ledsub_20/DOUT -> /led/ledsub_21/DIN
- R43 pad 2: /led/ledsub_21/DOUT -> /led/ledsub_22/DIN
- R45 pad 2: /led/ledsub_22/DOUT -> /led/ledsub_23/DIN
- R47 pad 2: /led/ledsub_23/DOUT -> /led/ledsub_18/DOUT
- R49 pad 2: /led/ledsub_24/DOUT -> /led/ledsub_19/DOUT
- U20 pad 5: /led/ledsub_20/DOUT -> /led/ledsub_19/DIN
- U21 pad 5: /led/ledsub_21/DOUT -> /led/ledsub_20/DIN
- U22 pad 5: /led/ledsub_22/DOUT -> /led/ledsub_21/DIN
- U23 pad 5: /led/ledsub_23/DOUT -> /led/ledsub_22/DIN
- U24 pad 5: /led/ledsub_24/DOUT -> /led/ledsub_23/DIN
Routing:
- net GND: track 111.6 -> 148.5 mm, vias 6 -> 10
- net +5V: track 105.5 -> 130.2 mm, vias 26 -> 31
- net /led/ledsub_20/DIN: track 0.00 -> 14.1 mm, vias 0 -> 2
- net /led/ledsub_23/DIN: track 0.00 -> 8.30 mm
- net /led/ledsub_22/DIN: track 0.00 -> 7.94 mm, vias 0 -> 2
- net /led/ledsub_23/DOUT: track 6.25 -> 0.00 mm
- net /led/ledsub_22/DOUT: track 5.12 -> 0.00 mm
- net /led/ledsub_18/DOUT: track 0.00 -> 4.48 mm
- net /led/ledsub_21/DIN: track 0.00 -> 4.27 mm
- net Net-(U19-DIN): track 0.00 -> 4.03 mm
- net Net-(U20-DIN): track 0.00 -> 2.69 mm
- net Net-(D14-B-): track 5.41 -> 7.63 mm
- net Net-(U19-VDD): track 3.61 -> 5.40 mm
- net /led/ledsub_21/DOUT: track 1.47 -> 0.00 mm
- net Net-(U21-DIN): track 0.00 -> 1.25 mm
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
Commit message: Zipp
Parts:
- moved R63 1.37 mm to (115.1, 102.2)
- moved R61 1.11 mm to (113.0, 102.6), turned to 0 degrees
- moved C33 0.20 mm to (124.0, 98.7)
Routing:
- net /led/ledsub_19/DOUT: track 0.00 -> 22.6 mm
- net +5V: track 130.2 -> 152.5 mm, vias 31 -> 35
- net GND: track 148.5 -> 154.6 mm, vias 10 -> 12
- net Net-(U32-DIN): track 0.00 -> 2.99 mm
- net Net-(U25-VDD): track 0.00 -> 2.42 mm
- net Net-(U21-VDD): track 0.00 -> 2.08 mm
- net /led/ledsub_31/DOUT: track 0.00 -> 2.01 mm
- net Net-(U25-DIN): track 0.00 -> 1.45 mm

Commit message: ABC
Parts:
- moved R71 5.83 mm to (139.7, 98.7), turned to 90 degrees
- moved C31 5.80 mm to (108.9, 100.2)
- moved C35 5.41 mm to (128.9, 101.5), turned to -90 degrees
- moved C36 5.31 mm to (133.4, 101.5), turned to -90 degrees
- moved C34 5.20 mm to (124.2, 101.0), turned to -90 degrees
- moved C32 5.04 mm to (116.0, 102.3), turned to -90 degrees
- moved C33 4.99 mm to (120.7, 102.3), turned to -90 degrees
- moved R63 4.88 mm to (119.5, 100.2), turned to 90 degrees
- moved R62 4.52 mm to (110.0, 100.1), turned to -90 degrees
- moved R65 4.28 mm to (124.2, 99.1), turned to -90 degrees
- moved R67 3.87 mm to (128.8, 99.7), turned to -90 degrees
- moved R69 3.72 mm to (133.3, 99.5), turned to -90 degrees
- moved R70 3.29 mm to (130.3, 102.0), turned to 180 degrees
- moved R72 3.18 mm to (135.0, 101.8), turned to 180 degrees
- moved R68 3.11 mm to (126.0, 101.9), turned to 180 degrees
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Connections:
- R61 pad 2: /led/ledsub_30/DOUT -> /led/ledsub_31/DIN
- R63 pad 2: /led/ledsub_31/DOUT -> /led/ledsub_32/DIN
- R65 pad 2: /led/ledsub_32/DOUT -> /led/ledsub_33/DIN
- R67 pad 2: /led/ledsub_33/DOUT -> /led/ledsub_34/DIN
- R69 pad 2: /led/ledsub_34/DOUT -> /led/ledsub_35/DIN
- R71 pad 2: /led/ledsub_35/DOUT -> /led/ledsub_30/DOUT
- U32 pad 5: /led/ledsub_32/DOUT -> /led/ledsub_31/DIN
- U33 pad 5: /led/ledsub_33/DOUT -> /led/ledsub_32/DIN
- U34 pad 5: /led/ledsub_34/DOUT -> /led/ledsub_33/DIN
- U35 pad 5: /led/ledsub_35/DOUT -> /led/ledsub_34/DIN
- U36 pad 5: /led/ledsub_36/DOUT -> /led/ledsub_35/DIN
Routing:
- net GND: track 154.6 -> 170.8 mm, vias 12 -> 16
- net +5V: track 152.5 -> 164.5 mm, vias 35 -> 42
- net Net-(U36-DIN): track 0.00 -> 5.78 mm
- net /led/ledsub_33/DIN: track 0.00 -> 5.13 mm, vias 0 -> 2
- net /led/ledsub_32/DIN: track 0.00 -> 4.72 mm, vias 0 -> 2
- net /led/ledsub_34/DIN: track 0.00 -> 4.70 mm, vias 0 -> 2
- net /led/ledsub_35/DIN: track 0.00 -> 4.31 mm
- net /led/ledsub_31/DIN: track 0.00 -> 4.25 mm
- net /led/ledsub_30/DOUT: track 0.00 -> 4.18 mm
- net Net-(U31-VDD): track 5.47 -> 2.14 mm
- net Net-(U33-DIN): track 0.00 -> 3.21 mm
- net Net-(U31-DIN): track 0.00 -> 3.21 mm
- net Net-(U34-DIN): track 0.00 -> 3.09 mm
- net Net-(U32-VDD): track 5.23 -> 2.17 mm
- net Net-(U35-DIN): track 0.00 -> 2.86 mm
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
Commit message: ABC
Routing:
- net +3.3V: track 12.4 -> 39.9 mm, vias 0 -> 2
- net /micro/RST: track 1.64 -> 23.2 mm
- net /micro/SWCLK: track 0.00 -> 11.7 mm
- net /micro/SWDIO: track 0.00 -> 11.5 mm
- net /led/DIN: track 36.2 -> 46.3 mm
- net GND: track 170.8 -> 177.3 mm
- net +5V: track 164.5 -> 166.4 mm, vias 42 -> 43

Commit message: Send
Parts:
- C41: footprint Capacitor_SMD:C_0201_0603Metric -> Capacitor_SMD:C_0805_2012Metric
- moved C41 1.99 mm to (96.3, 77.8)
- moved C40 1.10 mm to (94.5, 76.8)
- moved R33 0.61 mm to (127.3, 82.2), turned to -90 degrees
- moved R12 0.24 mm to (135.7, 62.9)
- moved R44 0.22 mm to (128.4, 84.5)
- moved R3 0.16 mm to (118.8, 61.5)
- moved R64 0.16 mm to (117.5, 102.0)
- moved C6 0.07 mm to (135.8, 65.0)
- moved C28 0.07 mm to (124.1, 94.8)
- moved R78 0.07 mm to (113.8, 61.5)
Routing:
- net /micro/RST: track 23.2 -> 26.5 mm
- net GND: track 177.3 -> 178.7 mm
- net +5V: track 166.4 -> 167.5 mm
- net Net-(U17-DIN): track 2.63 -> 3.67 mm
- net +3.3V: track 39.9 -> 40.8 mm
- net Net-(U6-VDD): track 5.02 -> 5.53 mm
