File: bizcard/bizcard.kicad_pcb (KiCad board)
At the start: 2 copper layers, 79.3 x 52.2 mm, 204 parts, among them J2 Conn_01x06_Pin, U1 MCP1700T-3302E_TT, U37 STM32F042K6Tx

Commit message: Grep
Parts:
- D1, D10, D11, D12, D13, D14, D15, D16, D17, D18, D19, D20, D21, D22, D23, D24, D25, D26, D27, D28, D29, D3, D30, D31, D32, D33, D34, D35, D36, D4, D40, D5, D6, D7, D8, D9: value ~ -> NH-B1212RGBA-HF
- U10, U11, U12, U13, U14, U15, U16, U17, U18, U19, U2, U20, U21, U22, U23, U24, U25, U26, U27, U28, U29, U3, U30, U31, U32, U33, U34, U35, U36, U38, U4, U5, U6, U7, U8, U9: value ~ -> WS2811F

Commit message: Drip
Parts:
- added C46: 100nF, Capacitor_SMD:C_0402_1005Metric, B.Cu at (94.5, 73.5)
- added Y1: SX7M8.192B10F20TN, Oscillator:Oscillator_SMD_SeikoEpson_SG8002CA-4Pin_7.0x5.0mm, B.Cu at (100.5, 74.0)
- C10, C11, C12, C13, C14, C15, C16, C17, C18, C19, C2, C20, C21, C22, C23, C24, C25, C26, C27, C28, C29, C3, C30, C31, C32, C33, C34, C35, C36, C4, C45, C5, C6, C7, C8, C9: value 100nF -> 1uF
Connections:
- U37 pad 2: unconnected-(U37-PF0-Pad2) -> /micro/CLK
Routing:
- net +3.3V: track 40.8 -> 54.7 mm, vias 2 -> 0
- net /micro/CLK: track 0.00 -> 9.86 mm
- net /micro/RST: track 26.5 -> 35.1 mm
- net GND: track 178.7 -> 181.0 mm
Other:
- board text added: "2. Navigate to"
- board text removed: "2. Follow instructions at"
- board text removed: "UWaterloo - Mechatronics '24"
