File: bizcard/led.kicad_sch (KiCad schematic)
At the start: 0 parts

Commit message: more
Changed lines of the file:
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@@
 	)
 	(sheet
-		(at 99.06 99.06)
+		(at 182.88 99.06)
 		(size 22.86 7.62)
 		(fields_autoplaced yes)
@@
 		)
 		(property "Sheetname" "ledsub_23"
-			(at 99.06 98.3484 0)
-			(effects
-				(font
-					(size 1.27 1.27)
-				)
-				(justify left bottom)
-			)
-		)
-		(property "Sheetfile" "ledsub.kicad_sch"
-			(at 99.06 107.2646 0)
-			(effects
-				(font
-					(size 1.27 1.27)
-				)
-				(justify left top)
-			)
-		)
-		(pin "DIN" input
-			(at 121.92 102.87 0)
-			(effects
-				(font
-					(size 1.27 1.27)
-				)
-				(justify right)
-			)
-		)
-		(pin "DOUT" output
-			(at 99.06 102.87 180)
+			(at 182.88 98.3484 0)
+			(effects
+				(font
+					(size 1.27 1.27)
+				)
+				(justify left bottom)
+			)
+		)
+		(property "Sheetfile" "ledsub.kicad_sch"
+			(at 182.88 107.2646 0)
+			(effects
+				(font
+					(size 1.27 1.27)
+				)
+				(justify left top)
+			)
+		)
+		(pin "DIN" input
+			(at 205.74 102.87 0)
+			(effects
+				(font
+					(size 1.27 1.27)
+				)
+				(justify right)
+			)
+		)
+		(pin "DOUT" output
+			(at 182.88 102.87 180)
 			(effects
 				(font
@@
 	)
 	(sheet
-		(at 212.09 99.06)
+		(at 68.58 99.06)
 		(size 22.86 7.62)
 		(fields_autoplaced yes)
@@
 		)
 		(property "Sheetname" "ledsub_19"
-			(at 212.09 98.3484 0)
-			(effects
-				(font
-					(size 1.27 1.27)
-				)
-				(justify left bottom)
-			)
-		)
-		(property "Sheetfile" "ledsub.kicad_sch"
-			(at 212.09 107.2646 0)
-			(effects
-				(font
-					(size 1.27 1.27)
-				)
-				(justify left top)
-			)
-		)
-		(pin "DIN" input
-			(at 234.95 102.87 0)
-			(effects
-				(font
-					(size 1.27 1.27)
-				)
-				(justify right)
-			)
-		)
-		(pin "DOUT" output
-			(at 212.09 102.87 180)
+			(at 68.58 98.3484 0)
+			(effects
+				(font
+					(size 1.27 1.27)
+				)
+				(justify left bottom)
+			)
+		)
+		(property "Sheetfile" "ledsub.kicad_sch"
+			(at 68.58 107.2646 0)
+			(effects
+				(font
+					(size 1.27 1.27)
+				)
+				(justify left top)
+			)
+		)
+		(pin "DIN" input
+			(at 91.44 102.87 0)
+			(effects
+				(font
+					(size 1.27 1.27)
+				)
+				(justify right)
+			)
+		)
+		(pin "DOUT" output
+			(at 68.58 102.87 180)
 			(effects
 				(font
@@
 	)
 	(sheet
-		(at 127 99.06)
+		(at 154.94 99.06)
 		(size 22.86 7.62)
 		(fields_autoplaced yes)
@@
 		)
 		(property "Sheetname" "ledsub_22"
-			(at 127 98.3484 0)
-			(effects
-				(font
-					(size 1.27 1.27)
-				)
-				(justify left bottom)
-			)
-		)
-		(property "Sheetfile" "ledsub.kicad_sch"
-			(at 127 107.2646 0)
-			(effects
-				(font
-					(size 1.27 1.27)
-				)
-				(justify left top)
-			)
-		)
-		(pin "DIN" input
-			(at 149.86 102.87 0)
-			(effects
-				(font
-					(size 1.27 1.27)
-				)
-				(justify right)
-			)
-		)
-		(pin "DOUT" output
-			(at 127 102.87 180)
+			(at 154.94 98.3484 0)
+			(effects
+				(font
+					(size 1.27 1.27)
+				)
+				(justify left bottom)
+			)
+		)
+		(property "Sheetfile" "ledsub.kicad_sch"
+			(at 154.94 107.2646 0)
+			(effects
+				(font
+					(size 1.27 1.27)
+				)
+				(justify left top)
+			)
+		)
+		(pin "DIN" input
+			(at 177.8 102.87 0)
+			(effects
+				(font
+					(size 1.27 1.27)
+				)
+				(justify right)
+			)
+		)
+		(pin "DOUT" output
+			(at 154.94 102.87 180)
 			(effects
 				(font
@@
 	)
 	(sheet
-		(at 154.94 99.06)
+		(at 127 99.06)
 		(size 22.86 7.62)
 		(fields_autoplaced yes)
@@
 		)
 		(property "Sheetname" "ledsub_21"
-			(at 154.94 98.3484 0)
-			(effects
-				(font
-					(size 1.27 1.27)
-				)
-				(justify left bottom)
-			)
-		)
-		(property "Sheetfile" "ledsub.kicad_sch"
-			(at 154.94 107.2646 0)
-			(effects
-				(font
-					(size 1.27 1.27)
-				)
-				(justify left top)
-			)
-		)
-		(pin "DIN" input
-			(at 177.8 102.87 0)
-			(effects
-				(font
-					(size 1.27 1.27)
-				)
-				(justify right)
-			)
-		)
-		(pin "DOUT" output
-			(at 154.94 102.87 180)
+			(at 127 98.3484 0)
+			(effects
+				(font
+					(size 1.27 1.27)
+				)
+				(justify left bottom)
+			)
+		)
+		(property "Sheetfile" "ledsub.kicad_sch"
+			(at 127 107.2646 0)
+			(effects
+				(font
+					(size 1.27 1.27)
+				)
+				(justify left top)
+			)
+		)
+		(pin "DIN" input
+			(at 149.86 102.87 0)
+			(effects
+				(font
+					(size 1.27 1.27)
+				)
+				(justify right)
+			)
+		)
+		(pin "DOUT" output
+			(at 127 102.87 180)
 			(effects
 				(font
@@
 	)
 	(sheet
-		(at 68.58 99.06)
+		(at 212.09 99.06)
 		(size 22.86 7.62)
 		(fields_autoplaced yes)
@@
 		)
 		(property "Sheetname" "ledsub_24"
-			(at 68.58 98.3484 0)
-			(effects
-				(font
-					(size 1.27 1.27)
-				)
-				(justify left bottom)
-			)
-		)
-		(property "Sheetfile" "ledsub.kicad_sch"
-			(at 68.58 107.2646 0)
-			(effects
-				(font
-					(size 1.27 1.27)
-				)
-				(justify left top)
-			)
-		)
-		(pin "DIN" input
-			(at 91.44 102.87 0)
-			(effects
-				(font
-					(size 1.27 1.27)
-				)
-				(justify right)
-			)
-		)
-		(pin "DOUT" output
-			(at 68.58 102.87 180)
+			(at 212.09 98.3484 0)
+			(effects
+				(font
+					(size 1.27 1.27)
+				)
+				(justify left bottom)
+			)
+		)
+		(property "Sheetfile" "ledsub.kicad_sch"
+			(at 212.09 107.2646 0)
+			(effects
+				(font
+					(size 1.27 1.27)
+				)
+				(justify left top)
+			)
+		)
+		(pin "DIN" input
+			(at 234.95 102.87 0)
+			(effects
+				(font
+					(size 1.27 1.27)
+				)
+				(justify right)
+			)
+		)
+		(pin "DOUT" output
+			(at 212.09 102.87 180)
 			(effects
 				(font
@@
 	)
 	(sheet
-		(at 182.88 99.06)
+		(at 99.06 99.06)
 		(size 22.86 7.62)
 		(fields_autoplaced yes)
@@
 		)
 		(property "Sheetname" "ledsub_20"
-			(at 182.88 98.3484 0)
-			(effects
-				(font
-					(size 1.27 1.27)
-				)
-				(justify left bottom)
-			)
-		)
-		(property "Sheetfile" "ledsub.kicad_sch"
-			(at 182.88 107.2646 0)
-			(effects
-				(font
-					(size 1.27 1.27)
-				)
-				(justify left top)
-			)
-		)
-		(pin "DIN" input
-			(at 205.74 102.87 0)
-			(effects
-				(font
-					(size 1.27 1.27)
-				)
-				(justify right)
-			)
-		)
-		(pin "DOUT" output
-			(at 182.88 102.87 180)
-			(effects
-				(font
+			(at 99.06 98.3484 0)
+			(effects
+				(font
+					(size 1.27 1.27)
+				)
+				(justify left bottom)
+			)
+		)
+		(property "Sheetfile" "ledsub.kicad_sch"
+			(at 99.06 107.2646 0)
+			(effects
+				(font
+					(size 1.27 1.27)
+				)
+				(justify left top)
+			)
+		)
+		(pin "DIN" input
+			(at 121.92 102.87 0)
+			(effects
+				(font
+					(size 1.27 1.27)
+				)
+				(justify right)
+			)
+		)
+		(pin "DOUT" output
+			(at 99.06 102.87 180)
+			(effects
+				(font

Commit message: ABC
Changed lines of the file:
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@@
 	)
 	(sheet
-		(at 154.94 132.08)
+		(at 127 132.08)
 		(size 22.86 7.62)
 		(fields_autoplaced yes)
@@
 		)
 		(property "Sheetname" "ledsub_33"
-			(at 154.94 131.3684 0)
-			(effects
-				(font
-					(size 1.27 1.27)
-				)
-				(justify left bottom)
-			)
-		)
-		(property "Sheetfile" "ledsub.kicad_sch"
-			(at 154.94 140.2846 0)
-			(effects
-				(font
-					(size 1.27 1.27)
-				)
-				(justify left top)
-			)
-		)
-		(pin "DIN" input
-			(at 177.8 135.89 0)
-			(effects
-				(font
-					(size 1.27 1.27)
-				)
-				(justify right)
-			)
-		)
-		(pin "DOUT" output
-			(at 154.94 135.89 180)
+			(at 127 131.3684 0)
+			(effects
+				(font
+					(size 1.27 1.27)
+				)
+				(justify left bottom)
+			)
+		)
+		(property "Sheetfile" "ledsub.kicad_sch"
+			(at 127 140.2846 0)
+			(effects
+				(font
+					(size 1.27 1.27)
+				)
+				(justify left top)
+			)
+		)
+		(pin "DIN" input
+			(at 149.86 135.89 0)
+			(effects
+				(font
+					(size 1.27 1.27)
+				)
+				(justify right)
+			)
+		)
+		(pin "DOUT" output
+			(at 127 135.89 180)
 			(effects
 				(font
@@
 	)
 	(sheet
-		(at 99.06 132.08)
+		(at 182.88 132.08)
 		(size 22.86 7.62)
 		(fields_autoplaced yes)
@@
 		)
 		(property "Sheetname" "ledsub_35"
-			(at 99.06 131.3684 0)
-			(effects
-				(font
-					(size 1.27 1.27)
-				)
-				(justify left bottom)
-			)
-		)
-		(property "Sheetfile" "ledsub.kicad_sch"
-			(at 99.06 140.2846 0)
-			(effects
-				(font
-					(size 1.27 1.27)
-				)
-				(justify left top)
-			)
-		)
-		(pin "DIN" input
-			(at 121.92 135.89 0)
-			(effects
-				(font
-					(size 1.27 1.27)
-				)
-				(justify right)
-			)
-		)
-		(pin "DOUT" output
-			(at 99.06 135.89 180)
+			(at 182.88 131.3684 0)
+			(effects
+				(font
+					(size 1.27 1.27)
+				)
+				(justify left bottom)
+			)
+		)
+		(property "Sheetfile" "ledsub.kicad_sch"
+			(at 182.88 140.2846 0)
+			(effects
+				(font
+					(size 1.27 1.27)
+				)
+				(justify left top)
+			)
+		)
+		(pin "DIN" input
+			(at 205.74 135.89 0)
+			(effects
+				(font
+					(size 1.27 1.27)
+				)
+				(justify right)
+			)
+		)
+		(pin "DOUT" output
+			(at 182.88 135.89 180)
 			(effects
 				(font
@@
 	)
 	(sheet
-		(at 127 132.08)
+		(at 154.94 132.08)
 		(size 22.86 7.62)
 		(fields_autoplaced yes)
@@
 		)
 		(property "Sheetname" "ledsub_34"
-			(at 127 131.3684 0)
-			(effects
-				(font
-					(size 1.27 1.27)
-				)
-				(justify left bottom)
-			)
-		)
-		(property "Sheetfile" "ledsub.kicad_sch"
-			(at 127 140.2846 0)
-			(effects
-				(font
-					(size 1.27 1.27)
-				)
-				(justify left top)
-			)
-		)
-		(pin "DIN" input
-			(at 149.86 135.89 0)
-			(effects
-				(font
-					(size 1.27 1.27)
-				)
-				(justify right)
-			)
-		)
-		(pin "DOUT" output
-			(at 127 135.89 180)
+			(at 154.94 131.3684 0)
+			(effects
+				(font
+					(size 1.27 1.27)
+				)
+				(justify left bottom)
+			)
+		)
+		(property "Sheetfile" "ledsub.kicad_sch"
+			(at 154.94 140.2846 0)
+			(effects
+				(font
+					(size 1.27 1.27)
+				)
+				(justify left top)
+			)
+		)
+		(pin "DIN" input
+			(at 177.8 135.89 0)
+			(effects
+				(font
+					(size 1.27 1.27)
+				)
+				(justify right)
+			)
+		)
+		(pin "DOUT" output
+			(at 154.94 135.89 180)
 			(effects
 				(font
@@
 	)
 	(sheet
-		(at 182.88 132.08)
+		(at 99.06 132.08)
 		(size 22.86 7.62)
 		(fields_autoplaced yes)
@@
 		)
 		(property "Sheetname" "ledsub_32"
-			(at 182.88 131.3684 0)
-			(effects
-				(font
-					(size 1.27 1.27)
-				)
-				(justify left bottom)
-			)
-		)
-		(property "Sheetfile" "ledsub.kicad_sch"
-			(at 182.88 140.2846 0)
-			(effects
-				(font
-					(size 1.27 1.27)
-				)
-				(justify left top)
-			)
-		)
-		(pin "DIN" input
-			(at 205.74 135.89 0)
-			(effects
-				(font
-					(size 1.27 1.27)
-				)
-				(justify right)
-			)
-		)
-		(pin "DOUT" output
-			(at 182.88 135.89 180)
+			(at 99.06 131.3684 0)
+			(effects
+				(font
+					(size 1.27 1.27)
+				)
+				(justify left bottom)
+			)
+		)
+		(property "Sheetfile" "ledsub.kicad_sch"
+			(at 99.06 140.2846 0)
+			(effects
+				(font
+					(size 1.27 1.27)
+				)
+				(justify left top)
+			)
+		)
+		(pin "DIN" input
+			(at 121.92 135.89 0)
+			(effects
+				(font
+					(size 1.27 1.27)
+				)
+				(justify right)
+			)
+		)
+		(pin "DOUT" output
+			(at 99.06 135.89 180)
 			(effects
 				(font
@@
 	)
 	(sheet
-		(at 212.09 132.08)
+		(at 68.58 132.08)
 		(size 22.86 7.62)
 		(fields_autoplaced yes)
@@
 		)
 		(property "Sheetname" "ledsub_31"
-			(at 212.09 131.3684 0)
-			(effects
-				(font
-					(size 1.27 1.27)
-				)
-				(justify left bottom)
-			)
-		)
-		(property "Sheetfile" "ledsub.kicad_sch"
-			(at 212.09 140.2846 0)
-			(effects
-				(font
-					(size 1.27 1.27)
-				)
-				(justify left top)
-			)
-		)
-		(pin "DIN" input
-			(at 234.95 135.89 0)
-			(effects
-				(font
-					(size 1.27 1.27)
-				)
-				(justify right)
-			)
-		)
-		(pin "DOUT" output
-			(at 212.09 135.89 180)
+			(at 68.58 131.3684 0)
+			(effects
+				(font
+					(size 1.27 1.27)
+				)
+				(justify left bottom)
+			)
+		)
+		(property "Sheetfile" "ledsub.kicad_sch"
+			(at 68.58 140.2846 0)
+			(effects
+				(font
+					(size 1.27 1.27)
+				)
+				(justify left top)
+			)
+		)
+		(pin "DIN" input
+			(at 91.44 135.89 0)
+			(effects
+				(font
+					(size 1.27 1.27)
+				)
+				(justify right)
+			)
+		)
+		(pin "DOUT" output
+			(at 68.58 135.89 180)
 			(effects
 				(font
@@
 	)
 	(sheet
-		(at 68.58 132.08)
+		(at 212.09 132.08)
 		(size 22.86 7.62)
 		(fields_autoplaced yes)
@@
 		)
 		(property "Sheetname" "ledsub_36"
-			(at 68.58 131.3684 0)
-			(effects
-				(font
-					(size 1.27 1.27)
-				)
-				(justify left bottom)
-			)
-		)
-		(property "Sheetfile" "ledsub.kicad_sch"
-			(at 68.58 140.2846 0)
-			(effects
-				(font
-					(size 1.27 1.27)
-				)
-				(justify left top)
-			)
-		)
-		(pin "DIN" input
-			(at 91.44 135.89 0)
-			(effects
-				(font
-					(size 1.27 1.27)
-				)
-				(justify right)
-			)
-		)
-		(pin "DOUT" output
-			(at 68.58 135.89 180)
-			(effects
-				(font
+			(at 212.09 131.3684 0)
+			(effects
+				(font
+					(size 1.27 1.27)
+				)
+				(justify left bottom)
+			)
+		)
+		(property "Sheetfile" "ledsub.kicad_sch"
+			(at 212.09 140.2846 0)
+			(effects
+				(font
+					(size 1.27 1.27)
+				)
+				(justify left top)
+			)
+		)
+		(pin "DIN" input
+			(at 234.95 135.89 0)
+			(effects
+				(font
+					(size 1.27 1.27)
+				)
+				(justify right)
+			)
+		)
+		(pin "DOUT" output
+			(at 212.09 135.89 180)
+			(effects
+				(font
