File: bizcard/_autosave-bizcard.kicad_pcb (KiCad board)
At the start: 2 copper layers, 79.6 x 52.5 mm, 204 parts, among them J2 Conn_01x06_Pin, U1 MCP1700T-3302E_TT, U37 STM32F042K6Tx

Commit message: Here
Other:
- board text added: "1. Plug in"
- board text added: "2. Follow instructions at"
- board text added: "OwenBrake.com/biz"
