File: bizcard/ledsub.kicad_sch (KiCad schematic)
At the start: 5 parts

Commit message: Push
Parts:
- renumbered C9 to C29, D9 to D12, R17 to R3, R18 to R58, U9 to U12
Changed lines of the file:
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@@
 		(on_board yes)
 		(dnp no)
-		(property "Reference" "R17"
+		(property "Reference" "R3"
 			(at 130.81 86.614 90)
 			(effects
@@
 		(dnp no)
 		(fields_autoplaced yes)
-		(property "Reference" "C9"
+		(property "Reference" "C29"
 			(at 151.13 86.3662 0)
 			(effects
@@
 		(dnp no)
 		(fields_autoplaced yes)
-		(property "Reference" "#PWR03"
+		(property "Reference" "#PWR0111"
 			(at 148.59 73.66 0)
 			(effects
@@
 		(dnp no)
 		(fields_autoplaced yes)
-		(property "Reference" "#PWR04"
+		(property "Reference" "#PWR0112"
 			(at 148.59 100.33 0)
 			(effects
@@
 		(dnp no)
 		(fields_autoplaced yes)
-		(property "Reference" "D9"
+		(property "Reference" "D12"
 			(at 111.76 67.9449 90)
 			(effects
@@
 		(dnp no)
 		(fields_autoplaced yes)
-		(property "Reference" "R18"
+		(property "Reference" "R58"
 			(at 151.13 76.1999 0)
 			(effects
@@
 		(dnp no)
 		(fields_autoplaced yes)
-		(property "Reference" "#PWR034"
+		(property "Reference" "#PWR046"
 			(at 109.22 99.06 0)
 			(effects
@@
 		(dnp no)
 		(fields_autoplaced yes)
-		(property "Reference" "U9"
+		(property "Reference" "U12"
 			(at 119.38 76.2 0)
 			(effects
@@
 		(dnp no)
 		(fields_autoplaced yes)
-		(property "Reference" "#PWR033"
+		(property "Reference" "#PWR045"
 			(at 104.14 58.42 0)
 			(effects

Commit message: dru
Parts:
- renumbered C29 to C30, D12 to D30, R3 to R59, R58 to R60, U12 to U30
Changed lines of the file:
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@@
 		(on_board yes)
 		(dnp no)
-		(property "Reference" "R3"
+		(property "Reference" "R59"
 			(at 130.81 86.614 90)
 			(effects
@@
 				(path "/7f3f26e1-61db-49d8-a68c-f315156bfd80/5d8cbbad-9a8a-47b9-976a-c32e026d92ff/87289c29-58df-42ab-a67e-edfae930b805"
 					(reference "R61")
+					(unit 1)
+				)
+				(path "/7f3f26e1-61db-49d8-a68c-f315156bfd80/5d8cbbad-9a8a-47b9-976a-c32e026d92ff/93c1b363-d575-4f58-b147-315e050d95c9"
+					(reference "R78")
 					(unit 1)
 				)
@@
 		(dnp no)
 		(fields_autoplaced yes)
-		(property "Reference" "C29"
+		(property "Reference" "C30"
 			(at 151.13 86.3662 0)
 			(effects
@@
 				(path "/7f3f26e1-61db-49d8-a68c-f315156bfd80/5d8cbbad-9a8a-47b9-976a-c32e026d92ff/87289c29-58df-42ab-a67e-edfae930b805"
 					(reference "C31")
+					(unit 1)
+				)
+				(path "/7f3f26e1-61db-49d8-a68c-f315156bfd80/5d8cbbad-9a8a-47b9-976a-c32e026d92ff/93c1b363-d575-4f58-b147-315e050d95c9"
+					(reference "C45")
 					(unit 1)
 				)
@@
 		(dnp no)
 		(fields_autoplaced yes)
-		(property "Reference" "#PWR0111"
+		(property "Reference" "#PWR079"
 			(at 148.59 73.66 0)
 			(effects
@@
 		(dnp no)
 		(fields_autoplaced yes)
-		(property "Reference" "#PWR0112"
+		(property "Reference" "#PWR080"
 			(at 148.59 100.33 0)
 			(effects
@@
 		(dnp no)
 		(fields_autoplaced yes)
-		(property "Reference" "D12"
+		(property "Reference" "D30"
 			(at 111.76 67.9449 90)
 			(effects
@@
 				(path "/7f3f26e1-61db-49d8-a68c-f315156bfd80/5d8cbbad-9a8a-47b9-976a-c32e026d92ff/87289c29-58df-42ab-a67e-edfae930b805"
 					(reference "D31")
+					(unit 1)
+				)
+				(path "/7f3f26e1-61db-49d8-a68c-f315156bfd80/5d8cbbad-9a8a-47b9-976a-c32e026d92ff/93c1b363-d575-4f58-b147-315e050d95c9"
+					(reference "D40")
 					(unit 1)
 				)
@@
 		(dnp no)
 		(fields_autoplaced yes)
-		(property "Reference" "R58"
+		(property "Reference" "R60"
 			(at 151.13 76.1999 0)
 			(effects
@@
 				(path "/7f3f26e1-61db-49d8-a68c-f315156bfd80/5d8cbbad-9a8a-47b9-976a-c32e026d92ff/87289c29-58df-42ab-a67e-edfae930b805"
 					(reference "R62")
+					(unit 1)
+				)
+				(path "/7f3f26e1-61db-49d8-a68c-f315156bfd80/5d8cbbad-9a8a-47b9-976a-c32e026d92ff/93c1b363-d575-4f58-b147-315e050d95c9"
+					(reference "R79")
 					(unit 1)
 				)
@@
 		(dnp no)
 		(fields_autoplaced yes)
-		(property "Reference" "#PWR046"
+		(property "Reference" "#PWR0118"
 			(at 109.22 99.06 0)
 			(effects
@@
 				(path "/7f3f26e1-61db-49d8-a68c-f315156bfd80/5d8cbbad-9a8a-47b9-976a-c32e026d92ff/87289c29-58df-42ab-a67e-edfae930b805"
 					(reference "#PWR0122")
+					(unit 1)
+				)
+				(path "/7f3f26e1-61db-49d8-a68c-f315156bfd80/5d8cbbad-9a8a-47b9-976a-c32e026d92ff/93c1b363-d575-4f58-b147-315e050d95c9"
+					(reference "#PWR0171")
 					(unit 1)
 				)
@@
 		(dnp no)
 		(fields_autoplaced yes)
-		(property "Reference" "U12"
+		(property "Reference" "U30"
 			(at 119.38 76.2 0)
 			(effects
@@
 				(path "/7f3f26e1-61db-49d8-a68c-f315156bfd80/5d8cbbad-9a8a-47b9-976a-c32e026d92ff/87289c29-58df-42ab-a67e-edfae930b805"
 					(reference "U31")
+					(unit 1)
+				)
+				(path "/7f3f26e1-61db-49d8-a68c-f315156bfd80/5d8cbbad-9a8a-47b9-976a-c32e026d92ff/93c1b363-d575-4f58-b147-315e050d95c9"
+					(reference "U38")
 					(unit 1)
 				)
@@
 		(dnp no)
 		(fields_autoplaced yes)
-		(property "Reference" "#PWR045"
+		(property "Reference" "#PWR0117"
 			(at 104.14 58.42 0)
 			(effects
@@
 					(unit 1)
 				)
+				(path "/7f3f26e1-61db-49d8-a68c-f315156bfd80/5d8cbbad-9a8a-47b9-976a-c32e026d92ff/93c1b363-d575-4f58-b147-315e050d95c9"
+					(reference "#PWR0172")
+					(unit 1)
+				)

Commit message: ABC
Parts:
- renumbered C30 to C9, D30 to D9, R59 to R17, R60 to R18, U30 to U9
Changed lines of the file:
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@@
 		(on_board yes)
 		(dnp no)
-		(property "Reference" "R59"
+		(property "Reference" "R17"
 			(at 130.81 86.614 90)
 			(effects
@@
 		(dnp no)
 		(fields_autoplaced yes)
-		(property "Reference" "C30"
+		(property "Reference" "C9"
 			(at 151.13 86.3662 0)
 			(effects
@@
 		(dnp no)
 		(fields_autoplaced yes)
-		(property "Reference" "#PWR079"
+		(property "Reference" "#PWR035"
 			(at 148.59 73.66 0)
 			(effects
@@
 		(dnp no)
 		(fields_autoplaced yes)
-		(property "Reference" "#PWR080"
+		(property "Reference" "#PWR036"
 			(at 148.59 100.33 0)
 			(effects
@@
 		(dnp no)
 		(fields_autoplaced yes)
-		(property "Reference" "D30"
+		(property "Reference" "D9"
 			(at 111.76 67.9449 90)
 			(effects
@@
 		(dnp no)
 		(fields_autoplaced yes)
-		(property "Reference" "R60"
+		(property "Reference" "R18"
 			(at 151.13 76.1999 0)
 			(effects
@@
 		(dnp no)
 		(fields_autoplaced yes)
-		(property "Reference" "#PWR0118"
+		(property "Reference" "#PWR034"
 			(at 109.22 99.06 0)
 			(effects
@@
 		(dnp no)
 		(fields_autoplaced yes)
-		(property "Reference" "U30"
+		(property "Reference" "U9"
 			(at 119.38 76.2 0)
 			(effects
@@
 		(dnp no)
 		(fields_autoplaced yes)
-		(property "Reference" "#PWR0117"
+		(property "Reference" "#PWR033"
 			(at 104.14 58.42 0)
 			(effects

Commit message: Send
Parts:
- renumbered C9 to C30, D9 to D30, R17 to R59, R18 to R60, U9 to U30
Changed lines of the file:
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@@
 		(on_board yes)
 		(dnp no)
-		(property "Reference" "R17"
+		(property "Reference" "R59"
 			(at 130.81 86.614 90)
 			(effects
@@
 		(dnp no)
 		(fields_autoplaced yes)
-		(property "Reference" "C9"
+		(property "Reference" "C30"
 			(at 151.13 86.3662 0)
 			(effects
@@
 		(dnp no)
 		(fields_autoplaced yes)
-		(property "Reference" "#PWR035"
+		(property "Reference" "#PWR079"
 			(at 148.59 73.66 0)
 			(effects
@@
 		(dnp no)
 		(fields_autoplaced yes)
-		(property "Reference" "#PWR036"
+		(property "Reference" "#PWR080"
 			(at 148.59 100.33 0)
 			(effects
@@
 		(dnp no)
 		(fields_autoplaced yes)
-		(property "Reference" "D9"
+		(property "Reference" "D30"
 			(at 111.76 67.9449 90)
 			(effects
@@
 		(dnp no)
 		(fields_autoplaced yes)
-		(property "Reference" "R18"
+		(property "Reference" "R60"
 			(at 151.13 76.1999 0)
 			(effects
@@
 		(dnp no)
 		(fields_autoplaced yes)
-		(property "Reference" "#PWR034"
+		(property "Reference" "#PWR0118"
 			(at 109.22 99.06 0)
 			(effects
@@
 		(dnp no)
 		(fields_autoplaced yes)
-		(property "Reference" "U9"
+		(property "Reference" "U30"
 			(at 119.38 76.2 0)
 			(effects
@@
 		(dnp no)
 		(fields_autoplaced yes)
-		(property "Reference" "#PWR033"
+		(property "Reference" "#PWR0117"
 			(at 104.14 58.42 0)
 			(effects

Commit message: Grep
Parts:
- D9: renamed from D30; value ~ -> NH-B1212RGBA-HF
- U9: renamed from U30; value ~ -> WS2811F
- renumbered C30 to C9, R59 to R17, R60 to R18
Changed lines of the file:
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@@
 		(on_board yes)
 		(dnp no)
-		(property "Reference" "R59"
+		(property "Reference" "R17"
 			(at 130.81 86.614 90)
 			(effects
@@
 		(dnp no)
 		(fields_autoplaced yes)
-		(property "Reference" "C30"
+		(property "Reference" "C9"
 			(at 151.13 86.3662 0)
 			(effects
@@
 		(dnp no)
 		(fields_autoplaced yes)
-		(property "Reference" "#PWR079"
+		(property "Reference" "#PWR035"
 			(at 148.59 73.66 0)
 			(effects
@@
 		(dnp no)
 		(fields_autoplaced yes)
-		(property "Reference" "#PWR080"
+		(property "Reference" "#PWR036"
 			(at 148.59 100.33 0)
 			(effects
@@
 		(dnp no)
 		(fields_autoplaced yes)
-		(property "Reference" "D30"
+		(property "Reference" "D9"
 			(at 111.76 67.9449 90)
 			(effects
@@
 			)
 		)
-		(property "Value" "~"
+		(property "Value" "NH-B1212RGBA-HF"
 			(at 111.76 69.85 90)
 			(effects
@@
 		(dnp no)
 		(fields_autoplaced yes)
-		(property "Reference" "R60"
+		(property "Reference" "R18"
 			(at 151.13 76.1999 0)
 			(effects
@@
 		(dnp no)
 		(fields_autoplaced yes)
-		(property "Reference" "#PWR0118"
+		(property "Reference" "#PWR034"
 			(at 109.22 99.06 0)
 			(effects
@@
 		(dnp no)
 		(fields_autoplaced yes)
-		(property "Reference" "U30"
+		(property "Reference" "U9"
 			(at 119.38 76.2 0)
 			(effects
@@
 			)
 		)
-		(property "Value" "~"
+		(property "Value" "WS2811F"
 			(at 119.38 78.74 0)
 			(effects
@@
 		(dnp no)
 		(fields_autoplaced yes)
-		(property "Reference" "#PWR0117"
+		(property "Reference" "#PWR033"
 			(at 104.14 58.42 0)
 			(effects

Commit message: Drip
Parts:
- C20: renamed from C9; value 100nF -> 1uF
- renumbered D9 to D20, R17 to R39, R18 to R40, U9 to U20
Changed lines of the file:
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@@
 		(on_board yes)
 		(dnp no)
-		(property "Reference" "R17"
+		(property "Reference" "R39"
 			(at 130.81 86.614 90)
 			(effects
@@
 		(dnp no)
 		(fields_autoplaced yes)
-		(property "Reference" "C9"
+		(property "Reference" "C20"
 			(at 151.13 86.3662 0)
 			(effects
@@
 			)
 		)
-		(property "Value" "100nF"
+		(property "Value" "1uF"
 			(at 151.13 88.9062 0)
 			(effects
@@
 		(dnp no)
 		(fields_autoplaced yes)
-		(property "Reference" "#PWR035"
+		(property "Reference" "#PWR079"
 			(at 148.59 73.66 0)
 			(effects
@@
 		(dnp no)
 		(fields_autoplaced yes)
-		(property "Reference" "#PWR036"
+		(property "Reference" "#PWR080"
 			(at 148.59 100.33 0)
 			(effects
@@
 		(dnp no)
 		(fields_autoplaced yes)
-		(property "Reference" "D9"
+		(property "Reference" "D20"
 			(at 111.76 67.9449 90)
 			(effects
@@
 		(dnp no)
 		(fields_autoplaced yes)
-		(property "Reference" "R18"
+		(property "Reference" "R40"
 			(at 151.13 76.1999 0)
 			(effects
@@
 		(dnp no)
 		(fields_autoplaced yes)
-		(property "Reference" "#PWR034"
+		(property "Reference" "#PWR078"
 			(at 109.22 99.06 0)
 			(effects
@@
 		(dnp no)
 		(fields_autoplaced yes)
-		(property "Reference" "U9"
+		(property "Reference" "U20"
 			(at 119.38 76.2 0)
 			(effects
@@
 		(dnp no)
 		(fields_autoplaced yes)
-		(property "Reference" "#PWR033"
+		(property "Reference" "#PWR077"
 			(at 104.14 58.42 0)
 			(effects
