File: bizcard/micro.kicad_sch (KiCad schematic)
At the start: 0 parts

Commit message: Push
Parts:
- added C1, C39, C40, C42: 100nF, Capacitor_SMD:C_0402_1005Metric, symbol Device:C_Small
- added C37, C38, C43: 1uF, Capacitor_SMD:C_0402_1005Metric, symbol Device:C_Small
- added C41: 4.7uF, Capacitor_SMD:C_0201_0603Metric, symbol Device:C_Small
- added C44: 4.7uF, Capacitor_SMD:C_0603_1608Metric, symbol Device:C_Small
- added D2, D38, D39: LED, LED_SMD:LED_0603_1608Metric, symbol Device:LED
- added D37: USBLC6-4SC6, digikey-footprints:SOT23-6L, symbol dk_TVS-Diodes:USBLC6-4SC6
- added J1: ~, USB:USB_PCBEDGE, symbol USB:USB
- added J2: Conn_01x06_Pin, Connector_PinHeader_2.54mm:PinHeader_1x06_P2.54mm_Vertical, symbol Connector:Conn_01x06_Pin
- added R1: 510Ω, Resistor_SMD:R_0603_1608Metric, symbol Device:R_US
- added R2: 220Ω, Resistor_SMD:R_0603_1608Metric, symbol Device:R_US
- added R73: 1kΩ, Resistor_SMD:R_0603_1608Metric, symbol Device:R_US
- added R74, R75, R76, R77: 0Ω, Resistor_SMD:R_0603_1608Metric, symbol Device:R_US
- added U1: MCP1700T-3302E_TT, digikey-footprints:SOT-23-3, symbol dk_PMIC-Voltage-Regulators-Linear:MCP1700T-3302E_TT
- added U37: STM32F042K6Tx, Package_QFP:LQFP-32_7x7mm_P0.8mm, symbol MCU_ST_STM32F0:STM32F042K6Tx
Connections:
- new net: R73.1, U37.29 (PB6)
- new net: D39.2 (A), R73.2
- new net: J1.1 (VBUS), R74.1
- new net: J1.2 (DM), R75.1
- new net: D37.1, R75.2
- new net: D38.2 (A), R2.2
- new net: D37.3, R76.2
- new net: J1.3 (DP), R76.1
- new net: J1.4 (GND), R77.1
- new net: D2.2 (A), R1.2
- new net +3.3V: C38.1, C40.1, C41.1, C42.1, C43.1, J2.1 (Pin_1), R2.1, U1.2 (OUT), U37.1 (VDD), U37.17 (VDDIO2), U37.5 (VDDA)
- new net +5V: C37.1, C39.1, C44.1, D37.5, J2.6 (Pin_6), R1.1, R74.2, U1.3 (IN)
- new net GND: C1.2, C37.2, C38.2, C39.2, C40.2, C41.2, C42.2, C43.2, C44.2, D2.1 (K), D37.2, D38.1 (K), D39.1 (K), J2.5 (Pin_5), R77.2, U1.1 (GND), U37.16 (VSS), U37.32 (VSSA)
- new net LED_DOUT: U37.13 (PA7)
- new net RST: C1.1, J2.4 (Pin_4), U37.4 (NRST)
- new net SWCLK: J2.3 (Pin_3), U37.24 (PA14)
- new net SWDIO: J2.2 (Pin_2), U37.23 (PA13)
- new net USB_DM: D37.6, U37.21 (PA11)
- new net USB_DP: D37.4, U37.22 (PA12)
Other:
- note added: "VDD"
- note added: "VDDA"
- note added: "VDDIO2"

Commit message: Send
Parts:
- C41: footprint Capacitor_SMD:C_0201_0603Metric -> Capacitor_SMD:C_0805_2012Metric
Changed lines of the file:
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@@
 			)
 		)
-		(property "Footprint" "Capacitor_SMD:C_0201_0603Metric"
+		(property "Footprint" "Capacitor_SMD:C_0805_2012Metric"
 			(at 217.17 53.34 0)
 			(effects

Commit message: Drip
Parts:
- added C46: 100nF, Capacitor_SMD:C_0402_1005Metric, symbol Device:C_Small
- added Y1: SX7M8.192B10F20TN, Oscillator:Oscillator_SMD_SeikoEpson_SG8002CA-4Pin_7.0x5.0mm, symbol Oscillator:SG-7050CAN
Connections:
- net +3.3V: now also C46.1, Y1.4 (VCC)
- net GND: now also C46.2, Y1.2 (GND)
- net CLK: now reaches U37.2 (PF0)
- net CLK: now also Y1.3 (OUT)
- no-connect marks 0 -> 20
Other:
- moved on the sheet: C1
